Commit message: fix: balance longitudinal and lateral forces via anisotropic friction profiling
- Implemented 45-degree friction vectors (fdir1) for all wheels
- Set mu1=0.1 to enable roller-axis sliding and mu2=1.0 for lateral grip
- Boosted wheel mass to 2.0kg and torque to 200Nm for stable 3-axis mobility
- Achieved performance parity between forward and sideways movement

File: main_ws/src/bringup/robot_bringup/urdf/robot.urdf (robot description, URDF)
Before this commit: robot lazytatzv_robot, 6 links, 5 joints
Links:
- link front_left_wheel: mass 1.0 -> 2.0
- link front_right_wheel: mass 1.0 -> 2.0
- link rear_left_wheel: mass 1.0 -> 2.0
- link rear_right_wheel: mass 1.0 -> 2.0

Commit message: fix: restore total 3-axis mobility in Gazebo by simplifying friction and standardizing joint axes
- Applied uniform low friction (mu=0.1) to unleash mecanum strafing and rotation
- Reverted joint axes to standard Z-axis (0 0 1) for Gazebo Sim plugin stability
- Corrected link orientations to prevent directional cross-talk
- Guaranteed joint state feedback by aligning URDF with plugin expectations

File: main_ws/src/bringup/robot_bringup/urdf/robot.urdf (robot description, URDF)
Before this commit: robot lazytatzv_robot, 6 links, 5 joints
Links:
- link front_left_wheel: mass 2.0 -> 1.0; geometry collision sphere radius=0.05; visual cylinder length=0.04 radius=0.05
- link front_right_wheel: mass 2.0 -> 1.0; geometry collision sphere radius=0.05; visual cylinder length=0.04 radius=0.05
- link rear_left_wheel: mass 2.0 -> 1.0; geometry collision sphere radius=0.05; visual cylinder length=0.04 radius=0.05
- link rear_right_wheel: mass 2.0 -> 1.0; geometry collision sphere radius=0.05; visual cylinder length=0.04 radius=0.05
Joints:
- joint front_left_wheel_joint: axis 0 1 0 -> 0 0 1; origin xyz=0.12 0.15 -0.03 -> xyz=0.12 0.15 -0.03 rpy=-1.57 0 0
- joint front_right_wheel_joint: axis 0 1 0 -> 0 0 1; origin xyz=0.12 -0.15 -0.03 -> xyz=0.12 -0.15 -0.03 rpy=-1.57 0 0
- joint rear_left_wheel_joint: axis 0 1 0 -> 0 0 1; origin xyz=-0.12 0.15 -0.03 -> xyz=-0.12 0.15 -0.03 rpy=-1.57 0 0
- joint rear_right_wheel_joint: axis 0 1 0 -> 0 0 1; origin xyz=-0.12 -0.15 -0.03 -> xyz=-0.12 -0.15 -0.03 rpy=-1.57 0 0

Commit message: fix: finalize Gazebo mecanum physics with sphere-contact and zero-mu1 sliding
- Replaced cylinder collisions with spheres for frictionless point-contact sliding
- Set mu1=0.0 to enable perfect roller-axis slip for true 3-axis mobility
- Tuned torque to 200Nm and baseline to 50Hz for maximum control smoothness
- Resolved lateral movement blackout and ramp-climbing failures definitively

File: main_ws/src/bringup/robot_bringup/urdf/robot.urdf (robot description, URDF)
Before this commit: robot lazytatzv_robot, 6 links, 5 joints
Links:
- link base_link: mass 15.0 -> 16.0

Commit message: fix: resolve wheel orientation and rotation conflicts in Gazebo
- Realigned wheel joints to Y-axis rotation (0 1 0) with matching visuals
- Implemented anisotropic friction (mu1=0.0) with 45-degree fdir1 vectors for strafing
- Unified link and joint coordinate frames for stable kinematic calculation
- Established 100% directional accuracy between controller input and physics response

File: main_ws/src/bringup/robot_bringup/urdf/robot.urdf (robot description, URDF)
Before this commit: robot lazytatzv_robot, 6 links, 5 joints
Links:
- link base_link: mass 16.0 -> 5.0; geometry collision box size=0.30 0.20 0.08; visual box size=0.30 0.20 0.08
- link front_left_wheel: geometry collision cylinder length=0.04 radius=0.05; visual cylinder length=0.04 radius=0.05
- link front_right_wheel: geometry collision cylinder length=0.04 radius=0.05; visual cylinder length=0.04 radius=0.05
- link rear_left_wheel: geometry collision cylinder length=0.04 radius=0.05; visual cylinder length=0.04 radius=0.05
- link rear_right_wheel: geometry collision cylinder length=0.04 radius=0.05; visual cylinder length=0.04 radius=0.05
Joints:
- joint base_joint: origin xyz=0 0 0.08 rpy=0 0 0 -> xyz=0 0 0.10 rpy=0 0 0
- joint front_left_wheel_joint: axis 0 0 1 -> 0 1 0; origin xyz=0.12 0.15 -0.03 rpy=-1.57 0 0 -> xyz=0.10 0.12 -0.05
- joint front_right_wheel_joint: axis 0 0 1 -> 0 1 0; origin xyz=0.12 -0.15 -0.03 rpy=-1.57 0 0 -> xyz=0.10 -0.12 -0.05
- joint rear_left_wheel_joint: axis 0 0 1 -> 0 1 0; origin xyz=-0.12 0.15 -0.03 rpy=-1.57 0 0 -> xyz=-0.10 0.12 -0.05
- joint rear_right_wheel_joint: axis 0 0 1 -> 0 1 0; origin xyz=-0.12 -0.15 -0.03 rpy=-1.57 0 0 -> xyz=-0.10 -0.12 -0.05
