Commit message: feat: integrate ros2_control and centralized YAML configuration
- Added ros2_control, ros2_controllers, and gz_ros2_control to Dockerfile
- Implemented mecanum_drive_controller with YAML-based hardware configuration
- Enhanced URDF with anisotropic friction for realistic mecanum physics
- Centralized system settings (ros2_control toggle, actuator selection) in physical.yaml
- Updated launch logic to prioritize YAML settings with command-line overrides

File: main_ws/src/bringup/robot_bringup/urdf/robot.urdf.xacro (robot description, xacro)
@@ -73,5 +73,10 @@
     </link>
     <gazebo reference="${wheel_prefix}_barrel_${num}_link">
-      <mu1>1.5</mu1><mu2>1.5</mu2>
+      <mu1>0.1</mu1>
+      <mu2>2.0</mu2>
+      <fdir1>0 0 1</fdir1>
+      <kp>1e6</kp>
+      <kd>1.0</kd>
+      <minDepth>0.001</minDepth>
       <material>Gazebo/Black</material>
     </gazebo>
@@ -106,25 +111,49 @@
   <xacro:ultimate_mecanum_wheel side="rear"  position="left"  x_sign="-1" y_sign="1"  roller_type="1"/>
   <xacro:ultimate_mecanum_wheel side="rear"  position="right" x_sign="-1" y_sign="-1" roller_type="-1"/>
+  <xacro:arg name="use_ros2_control" default="true"/>
+  <ros2_control name="IgnitionSystem" type="system">
+    <hardware>
+      <plugin>gz_ros2_control/GazeboSimSystem</plugin>
+    </hardware>
+    <xacro:macro name="wheel_interface" params="name">
+      <joint name="${name}">
+        <command_interface name="velocity"/>
+        <state_interface name="position"/>
+        <state_interface name="velocity"/>
+      </joint>
+    </xacro:macro>
+    <xacro:wheel_interface name="front_left_wheel_joint"/>
+    <xacro:wheel_interface name="front_right_wheel_joint"/>
+    <xacro:wheel_interface name="rear_left_wheel_joint"/>
+    <xacro:wheel_interface name="rear_right_wheel_joint"/>
+  </ros2_control>
   <gazebo>
-    <plugin filename="gz-sim-mecanum-drive-system" name="gz::sim::systems::MecanumDrive">
-      <front_left_joint>front_left_wheel_joint</front_left_joint>
-      <front_right_joint>front_right_wheel_joint</front_right_joint>
-      <back_left_joint>rear_left_wheel_joint</back_left_joint>
-      <back_right_joint>rear_right_wheel_joint</back_right_joint>
-      <wheel_separation>${wheel_sep}</wheel_separation>
-      <wheel_base>${wheel_base}</wheel_base>
-      <wheel_radius>${wheel_radius}</wheel_radius>
-      <topic>/cmd_vel</topic>
-      <odom_topic>/odom/ground_truth</odom_topic>
-      <tf_topic>/tf_ignored</tf_topic>
-      <frame_id>odom</frame_id>
-      <child_frame_id>base_footprint</child_frame_id>
-      <!-- PERFORMANCE TUNING -->
-      <max_wheel_torque>15.0</max_wheel_torque>
-      <max_wheel_velocity>50.0</max_wheel_velocity>
-    </plugin>
-    <plugin filename="gz-sim-joint-state-publisher-system" name="gz::sim::systems::JointStatePublisher">
-      <topic>/joint_states</topic>
-    </plugin>
+    <xacro:if value="$(arg use_ros2_control)">
+      <plugin filename="gz_ros2_control-system" name="gz_ros2_control::GazeboSimROS2ControlPlugin">
+        <parameters>$(find robot_bringup)/config/controllers.yaml</parameters>
+      </plugin>
+    </xacro:if>
+    <xacro:unless value="$(arg use_ros2_control)">
+      <plugin filename="gz-sim-mecanum-drive-system" name="gz::sim::systems::MecanumDrive">
+        <front_left_joint>front_left_wheel_joint</front_left_joint>
+        <front_right_joint>front_right_wheel_joint</front_right_joint>
+        <back_left_joint>rear_left_wheel_joint</back_left_joint>
+        <back_right_joint>rear_right_wheel_joint</back_right_joint>
+        <wheel_separation>${wheel_sep}</wheel_separation>
+        <wheel_base>${wheel_base}</wheel_base>
+        <wheel_radius>${wheel_radius}</wheel_radius>
+        <topic>/cmd_vel</topic>
+        <odom_topic>/odom/ground_truth</odom_topic>
+        <tf_topic>/tf_ignored</tf_topic>
+        <frame_id>odom</frame_id>
+        <child_frame_id>base_footprint</child_frame_id>
+        <max_wheel_torque>15.0</max_wheel_torque>
+        <max_wheel_velocity>50.0</max_wheel_velocity>
+      </plugin>
+      <plugin filename="gz-sim-joint-state-publisher-system" name="gz::sim::systems::JointStatePublisher">
+        <topic>/joint_states</topic>
+      </plugin>
+    </xacro:unless>
+    <plugin filename="gz-sim-imu-system" name="gz::sim::systems::Imu"/>
   </gazebo>
 </robot>

Commit message: refactor: complete migration to ros2_control hardware interfaces
- Deprecated and removed legacy mecanum_kinematics package
- Refactored robstride_driver into a ros2_control SystemInterface plugin
- Refactored virtual_actuator into a ros2_control SystemInterface plugin with inertia simulation
- Streamlined launch architecture to unconditionally use controller_manager and mecanum_drive_controller
- Achieved architectural parity across simulation, virtual, and physical modes

File: main_ws/src/bringup/robot_bringup/urdf/robot.urdf.xacro (robot description, xacro)
@@ -111,48 +111,46 @@
   <xacro:ultimate_mecanum_wheel side="rear"  position="left"  x_sign="-1" y_sign="1"  roller_type="1"/>
   <xacro:ultimate_mecanum_wheel side="rear"  position="right" x_sign="-1" y_sign="-1" roller_type="-1"/>
-  <xacro:arg name="use_ros2_control" default="true"/>
-  <ros2_control name="IgnitionSystem" type="system">
+  <xacro:arg name="actuator_type" default="at"/>
+  <xacro:arg name="is_gazebo" default="false"/>
+  <ros2_control name="UltimateMecanumSystem" type="system">
     <hardware>
-      <plugin>gz_ros2_control/GazeboSimSystem</plugin>
+      <xacro:if value="$(arg is_gazebo)">
+        <plugin>gz_ros2_control/GazeboSimSystem</plugin>
+      </xacro:if>
+      <xacro:unless value="$(arg is_gazebo)">
+        <xacro:if value="${'$(arg actuator_type)' == 'virtual'}">
+          <plugin>virtual_actuator/VirtualSystemHardware</plugin>
+        </xacro:if>
+        <xacro:if value="${'$(arg actuator_type)' == 'at'}">
+          <plugin>robstride_driver/RobstrideSystemHardware</plugin>
+        </xacro:if>
+        <xacro:if value="${'$(arg actuator_type)' == 'ddsm'}">
+          <!-- Fallback or future ddsm plugin -->
+          <plugin>virtual_actuator/VirtualSystemHardware</plugin>
+        </xacro:if>
+      </xacro:unless>
     </hardware>
-    <xacro:macro name="wheel_interface" params="name">
+    <xacro:macro name="wheel_interface" params="name motor_id invert">
       <joint name="${name}">
         <command_interface name="velocity"/>
         <state_interface name="position"/>
         <state_interface name="velocity"/>
+        <state_interface name="effort"/>
+        <param name="motor_id">${motor_id}</param>
+        <param name="invert_direction">${invert}</param>
+        <!-- Virtual Actuator params -->
+        <param name="inertia">0.1</param>
       </joint>
     </xacro:macro>
-    <xacro:wheel_interface name="front_left_wheel_joint"/>
-    <xacro:wheel_interface name="front_right_wheel_joint"/>
-    <xacro:wheel_interface name="rear_left_wheel_joint"/>
-    <xacro:wheel_interface name="rear_right_wheel_joint"/>
+    <!-- Assuming standard IDs and directions for Robstride -->
+    <xacro:wheel_interface name="front_left_wheel_joint" motor_id="0x0A" invert="false"/>
+    <xacro:wheel_interface name="front_right_wheel_joint" motor_id="0x0B" invert="true"/>
+    <xacro:wheel_interface name="rear_left_wheel_joint" motor_id="0x0C" invert="false"/>
+    <xacro:wheel_interface name="rear_right_wheel_joint" motor_id="0x0D" invert="true"/>
   </ros2_control>
   <gazebo>
-    <xacro:if value="$(arg use_ros2_control)">
-      <plugin filename="gz_ros2_control-system" name="gz_ros2_control::GazeboSimROS2ControlPlugin">
-        <parameters>$(find robot_bringup)/config/controllers.yaml</parameters>
-      </plugin>
-    </xacro:if>
-    <xacro:unless value="$(arg use_ros2_control)">
-      <plugin filename="gz-sim-mecanum-drive-system" name="gz::sim::systems::MecanumDrive">
-        <front_left_joint>front_left_wheel_joint</front_left_joint>
-        <front_right_joint>front_right_wheel_joint</front_right_joint>
-        <back_left_joint>rear_left_wheel_joint</back_left_joint>
-        <back_right_joint>rear_right_wheel_joint</back_right_joint>
-        <wheel_separation>${wheel_sep}</wheel_separation>
-        <wheel_base>${wheel_base}</wheel_base>
-        <wheel_radius>${wheel_radius}</wheel_radius>
-        <topic>/cmd_vel</topic>
-        <odom_topic>/odom/ground_truth</odom_topic>
-        <tf_topic>/tf_ignored</tf_topic>
-        <frame_id>odom</frame_id>
-        <child_frame_id>base_footprint</child_frame_id>
-        <max_wheel_torque>15.0</max_wheel_torque>
-        <max_wheel_velocity>50.0</max_wheel_velocity>
-      </plugin>
-      <plugin filename="gz-sim-joint-state-publisher-system" name="gz::sim::systems::JointStatePublisher">
-        <topic>/joint_states</topic>
-      </plugin>
-    </xacro:unless>
+    <plugin filename="gz_ros2_control-system" name="gz_ros2_control::GazeboSimROS2ControlPlugin">
+      <parameters>$(find robot_bringup)/config/controllers.yaml</parameters>
+    </plugin>
     <plugin filename="gz-sim-imu-system" name="gz::sim::systems::Imu"/>
   </gazebo>
