Commit message: feat: プロフェッショナルな Config-Driven アーキテクチャの実装とベンチテスト環境の構築
- Config-Driven: 物理特性、ハードウェア設定、制御ゲインを YAML に集約し Single Source of Truth を実現
- URDF動的化: xacro:load_yaml を導入し、物理モデルを YAML から自動生成
- 制御ノード最適化: imu_stabilizer の全ゲインを ROS 2 パラメータ化し、動的チューニングに対応
- ベンチテスト環境: モーター1軸の徹底解析を可能にする 1軸専用URDF/コントローラーおよび make bench コマンドを追加
- 解析ワークフローの統合: シグナル注入先をベンチ用コントローラーにも対応

File: main_ws/src/bringup/robot_bringup/urdf/robot.urdf.xacro (robot description, xacro)
@@ -4,35 +4,42 @@
   <xacro:include filename="$(find robot_bringup)/urdf/include/common.xacro"/>
   <xacro:include filename="$(find robot_bringup)/urdf/include/wheel.xacro"/>
-  <!-- 2. Properties -->
-  <xacro:property name="base_mass"    value="18.0"/>
-  <xacro:property name="hub_mass"     value="0.5"/>
-  <xacro:property name="wheel_radius" value="0.05"/>
-  <xacro:property name="wheel_base"   value="0.40"/>
-  <xacro:property name="wheel_sep"    value="0.40"/>
+  <!-- 2. Dynamic Configuration from YAML -->
+  <xacro:property name="props" value="${xacro.load_yaml('$(find robot_bringup)/config/params/physical_props.yaml')}"/>
+  <xacro:property name="hw"    value="${xacro.load_yaml('$(find robot_bringup)/config/params/hardware_config.yaml')}"/>
+  <!-- Physical Specs -->
+  <xacro:property name="base_mass"    value="${props['base']['mass']}"/>
+  <xacro:property name="base_w"       value="${props['base']['width']}"/>
+  <xacro:property name="base_l"       value="${props['base']['length']}"/>
+  <xacro:property name="base_h"       value="${props['base']['height']}"/>
+  <xacro:property name="hub_mass"     value="${props['wheels']['mass']}"/>
+  <xacro:property name="wheel_radius" value="${props['wheels']['radius']}"/>
+  <xacro:property name="wheel_base"   value="${props['wheels']['wheel_base']}"/>
+  <xacro:property name="wheel_sep"    value="${props['wheels']['track_width']}"/>
   <!-- 3. Base Body -->
   <link name="base_footprint"/>
   <link name="base_link">
-    <xacro:box_inertia m="${base_mass}" w="0.5" h="0.5" d="0.1"/>
-    <visual name="base_vis"><origin xyz="0 0 0.05"/><geometry><box size="0.45 0.45 0.1"/></geometry><material name="black"/></visual>
-    <collision name="base_col"><origin xyz="0 0 0.05"/><geometry><box size="0.45 0.45 0.1"/></geometry></collision>
+    <xacro:box_inertia m="${base_mass}" w="${base_w}" h="${base_l}" d="${base_h}"/>
+    <visual name="base_vis"><origin xyz="0 0 0.05"/><geometry><box size="${base_w - 0.05} ${base_l - 0.05} ${base_h}"/></geometry><material name="black"/></visual>
+    <collision name="base_col"><origin xyz="0 0 0.05"/><geometry><box size="${base_w - 0.05} ${base_l - 0.05} ${base_h}"/></geometry></collision>
   </link>
   <joint name="base_joint" type="fixed"><parent link="base_footprint"/><child link="base_link"/><origin xyz="0 0 0.05"/></joint>
   <!-- 4. Sensors -->
-  <!-- IMU -->
+  <xacro:property name="imu_o" value="${props['sensors']['imu_offset']}"/>
   <link name="imu_link"><xacro:box_inertia m="0.01" w="0.01" h="0.01" d="0.01" oz="0"/></link>
-  <joint name="imu_joint" type="fixed"><parent link="base_link"/><child link="imu_link"/><origin xyz="0 0 0.1"/></joint>
-  <gazebo reference="imu_link"><sensor name="imu_sensor" type="imu"><always_on>1</always_on><update_rate>100</update_rate><topic>imu</topic></sensor></gazebo>
-  <!-- Camera -->
+  <joint name="imu_joint" type="fixed"><parent link="base_link"/><child link="imu_link"/><origin xyz="${imu_o['x']} ${imu_o['y']} ${imu_o['z']}"/></joint>
+  <xacro:property name="cam_o" value="${props['sensors']['camera_offset']}"/>
   <link name="camera_link"><visual name="cam_vis"><geometry><box size="0.02 0.05 0.02"/></geometry><material name="black"/></visual></link>
-  <joint name="camera_joint" type="fixed"><parent link="base_link"/><child link="camera_link"/><origin xyz="0.2 0 0.1" rpy="0 0.2 0"/></joint>
-  <gazebo reference="camera_link"><sensor name="main_camera" type="camera"><always_on>1</always_on><update_rate>20</update_rate><topic>camera/image_raw</topic><camera><horizontal_fov>1.396</horizontal_fov><image><width>640</width><height>480</height><format>R8G8B8</format></image><clip><near>0.05</near><far>10.0</far></clip></camera></sensor></gazebo>
+  <joint name="camera_joint" type="fixed"><parent link="base_link"/><child link="camera_link"/><origin xyz="${cam_o['x']} ${cam_o['y']} ${cam_o['z']}" rpy="${cam_o['roll']} ${cam_o['pitch']} ${cam_o['yaw']}"/></joint>
   <!-- 5. Actuators (Wheels) -->
-  <xacro:mecanum_wheel name="front_left"  x="0.2"  y="0.2" roller_type="-1" hub_mass="${hub_mass}" wheel_radius="${wheel_radius}"/>
-  <xacro:mecanum_wheel name="front_right" x="0.2"  y="-0.2" roller_type="1"  hub_mass="${hub_mass}" wheel_radius="${wheel_radius}"/>
-  <xacro:mecanum_wheel name="rear_left"   x="-0.2" y="0.2"  roller_type="1"  hub_mass="${hub_mass}" wheel_radius="${wheel_radius}"/>
-  <xacro:mecanum_wheel name="rear_right"  x="-0.2" y="-0.2" roller_type="-1" hub_mass="${hub_mass}" wheel_radius="${wheel_radius}"/>
+  <xacro:property name="off_x" value="${wheel_base / 2.0}"/>
+  <xacro:property name="off_y" value="${wheel_sep / 2.0}"/>
+  <xacro:mecanum_wheel name="front_left"  x="${off_x}"  y="${off_y}" roller_type="-1" hub_mass="${hub_mass}" wheel_radius="${wheel_radius}"/>
+  <xacro:mecanum_wheel name="front_right" x="${off_x}"  y="${-off_y}" roller_type="1"  hub_mass="${hub_mass}" wheel_radius="${wheel_radius}"/>
+  <xacro:mecanum_wheel name="rear_left"   x="${-off_x}" y="${off_y}"  roller_type="1"  hub_mass="${hub_mass}" wheel_radius="${wheel_radius}"/>
+  <xacro:mecanum_wheel name="rear_right"  x="${-off_x}" y="${-off_y}" roller_type="-1" hub_mass="${hub_mass}" wheel_radius="${wheel_radius}"/>
   <!-- 6. ros2_control & Gazebo -->
   <xacro:arg name="gazebo" default="false"/>
-  <xacro:arg name="usb_path" default="/dev/ttyUSB0"/>
+  <xacro:arg name="usb_path" default="${hw['hardware']['usb_port']}"/>
+  <xacro:arg name="bench_mode" default="false"/>
   <ros2_control name="BaseKitSystem" type="system">
     <hardware>
@@ -43,25 +50,34 @@
         <plugin>robstride_driver/RobstrideSystemHardware</plugin>
         <param name="usb_path">$(arg usb_path)</param>
-        <param name="protocol">at</param>
-        <param name="serial_baud">115200</param>
+        <param name="protocol">${hw['hardware']['protocol']}</param>
+        <param name="serial_baud">${hw['hardware']['baud_rate']}</param>
       </xacro:unless>
     </hardware>
-    <xacro:macro name="joint_if" params="name id">
-      <joint name="${name}_wheel_joint">
-        <command_interface name="velocity">
-          <param name="p">40.0</param>
-          <param name="i">1.0</param>
-          <param name="d">1.0</param>
-        </command_interface>
+    <xacro:if value="$(arg bench_mode)">
+      <joint name="bench_joint">
+        <command_interface name="velocity"><param name="p">40.0</param></command_interface>
         <state_interface name="position"/><state_interface name="velocity"/><state_interface name="effort"/>
-        <param name="motor_id">${id}</param>
+        <param name="motor_id">${hw['hardware']['motors']['bench_id']}</param>
         <param name="invert_direction">false</param>
       </joint>
-    </xacro:macro>
-    <xacro:joint_if name="front_left" id="1"/>
-    <xacro:joint_if name="front_right" id="2"/>
-    <xacro:joint_if name="rear_left" id="3"/>
-    <xacro:joint_if name="rear_right" id="4"/>
+    </xacro:if>
+    <xacro:unless value="$(arg bench_mode)">
+      <xacro:macro name="joint_if" params="name hw_node">
+        <joint name="${name}_wheel_joint">
+          <command_interface name="velocity">
+            <param name="p">40.0</param><param name="i">1.0</param><param name="d">1.0</param>
+          </command_interface>
+          <state_interface name="position"/><state_interface name="velocity"/><state_interface name="effort"/>
+          <param name="motor_id">${hw['hardware']['motors'][hw_node]['id']}</param>
+          <param name="invert_direction">${hw['hardware']['motors'][hw_node]['invert']}</param>
+        </joint>
+      </xacro:macro>
+      <xacro:joint_if name="front_left"  hw_node="front_left"/>
+      <xacro:joint_if name="front_right" hw_node="front_right"/>
+      <xacro:joint_if name="rear_left"   hw_node="rear_left"/>
+      <xacro:joint_if name="rear_right"  hw_node="rear_right"/>
+    </xacro:unless>
   </ros2_control>
+...
   <gazebo>
     <plugin filename="gz_ros2_control-system" name="gz_ros2_control::GazeboSimROS2ControlPlugin">

Commit message: Fix URDF bugs: correct x/y box size mapping, swap width/length, add visuals for camera and imu

File: main_ws/src/bringup/robot_bringup/urdf/robot.urdf.xacro (robot description, xacro)
@@ -20,15 +20,28 @@
   <link name="base_link">
     <xacro:box_inertia m="${base_mass}" w="${base_w}" h="${base_l}" d="${base_h}"/>
-    <visual name="base_vis"><origin xyz="0 0 0.05"/><geometry><box size="${base_w - 0.05} ${base_l - 0.05} ${base_h}"/></geometry><material name="black"/></visual>
-    <collision name="base_col"><origin xyz="0 0 0.05"/><geometry><box size="${base_w - 0.05} ${base_l - 0.05} ${base_h}"/></geometry></collision>
+    <visual name="base_vis"><origin xyz="0 0 0.05"/><geometry><box size="${base_l} ${base_w} ${base_h}"/></geometry><material name="black"/></visual>
+    <collision name="base_col"><origin xyz="0 0 0.05"/><geometry><box size="${base_l} ${base_w} ${base_h}"/></geometry></collision>
   </link>
   <joint name="base_joint" type="fixed"><parent link="base_footprint"/><child link="base_link"/><origin xyz="0 0 0.05"/></joint>
   <!-- 4. Sensors -->
   <xacro:property name="imu_o" value="${props['sensors']['imu_offset']}"/>
-  <link name="imu_link"><xacro:box_inertia m="0.01" w="0.01" h="0.01" d="0.01" oz="0"/></link>
+  <link name="imu_link">
+    <xacro:box_inertia m="0.01" w="0.01" h="0.01" d="0.01" oz="0"/>
+    <visual name="imu_vis"><geometry><box size="0.03 0.03 0.01"/></geometry><material name="red"/></visual>
+  </link>
   <joint name="imu_joint" type="fixed"><parent link="base_link"/><child link="imu_link"/><origin xyz="${imu_o['x']} ${imu_o['y']} ${imu_o['z']}"/></joint>
   <xacro:property name="cam_o" value="${props['sensors']['camera_offset']}"/>
-  <link name="camera_link"><visual name="cam_vis"><geometry><box size="0.02 0.05 0.02"/></geometry><material name="black"/></visual></link>
+  <link name="camera_link">
+    <xacro:box_inertia m="0.01" w="0.02" h="0.05" d="0.02"/>
+    <visual name="cam_vis"><geometry><box size="0.02 0.05 0.02"/></geometry><material name="red"/></visual>
+  </link>
   <joint name="camera_joint" type="fixed"><parent link="base_link"/><child link="camera_link"/><origin xyz="${cam_o['x']} ${cam_o['y']} ${cam_o['z']}" rpy="${cam_o['roll']} ${cam_o['pitch']} ${cam_o['yaw']}"/></joint>
+  <!-- Camera Optical Frame -->
+  <link name="camera_link_optical"/>
+  <joint name="camera_optical_joint" type="fixed">
+    <parent link="camera_link"/>
+    <child link="camera_link_optical"/>
+    <origin xyz="0 0 0" rpy="-1.570796 0 -1.570796"/>
+  </joint>
   <!-- 5. Actuators (Wheels) -->
   <xacro:property name="off_x" value="${wheel_base / 2.0}"/>
@@ -116,3 +129,24 @@
     </sensor>
   </gazebo>
+  <!-- Gazebo Camera Sensor Plugin -->
+  <gazebo reference="camera_link">
+    <sensor name="camera_sensor" type="camera">
+      <always_on>true</always_on>
+      <update_rate>30.0</update_rate>
+      <topic>/camera/image_raw</topic>
+      <gz_frame_id>camera_link_optical</gz_frame_id>
+      <camera>
+        <horizontal_fov>1.047198</horizontal_fov>
+        <image>
+          <width>640</width>
+          <height>480</height>
+          <format>R8G8B8</format>
+        </image>
+        <clip>
+          <near>0.05</near>
+          <far>8.0</far>
+        </clip>
+      </camera>
+    </sensor>
+  </gazebo>
 </robot>

Commit message: Revert base_link visual/collision origin shift to fix camera position

File: main_ws/src/bringup/robot_bringup/urdf/robot.urdf.xacro (robot description, xacro)
@@ -23,5 +23,5 @@
     <collision name="base_col"><origin xyz="0 0 0.05"/><geometry><box size="${base_l} ${base_w} ${base_h}"/></geometry></collision>
   </link>
-  <joint name="base_joint" type="fixed"><parent link="base_footprint"/><child link="base_link"/><origin xyz="0 0 ${wheel_radius}"/></joint>
+  <joint name="base_joint" type="fixed"><parent link="base_footprint"/><child link="base_link"/><origin xyz="0 0 0.05"/></joint>
   <!-- 4. Sensors -->
   <xacro:property name="imu_o" value="${props['sensors']['imu_offset']}"/>
@@ -47,8 +47,8 @@
   <xacro:property name="off_x" value="${wheel_base / 2.0}"/>
   <xacro:property name="off_y" value="${wheel_sep / 2.0}"/>
-  <xacro:mecanum_wheel name="front_left"  x="${off_x}"  y="${off_y}" roller_type="-1" hub_mass="${hub_mass}" wheel_radius="${wheel_radius}"/>
-  <xacro:mecanum_wheel name="front_right" x="${off_x}"  y="${-off_y}" roller_type="1"  hub_mass="${hub_mass}" wheel_radius="${wheel_radius}"/>
-  <xacro:mecanum_wheel name="rear_left"   x="${-off_x}" y="${off_y}"  roller_type="1"  hub_mass="${hub_mass}" wheel_radius="${wheel_radius}"/>
-  <xacro:mecanum_wheel name="rear_right"  x="${-off_x}" y="${-off_y}" roller_type="-1" hub_mass="${hub_mass}" wheel_radius="${wheel_radius}"/>
+  <xacro:mecanum_wheel name="front_left"  x="${off_x}"  y="${off_y}" roller_type="1" hub_mass="${hub_mass}" wheel_radius="${wheel_radius}"/>
+  <xacro:mecanum_wheel name="front_right" x="${off_x}"  y="${-off_y}" roller_type="-1"  hub_mass="${hub_mass}" wheel_radius="${wheel_radius}"/>
+  <xacro:mecanum_wheel name="rear_left"   x="${-off_x}" y="${off_y}"  roller_type="-1"  hub_mass="${hub_mass}" wheel_radius="${wheel_radius}"/>
+  <xacro:mecanum_wheel name="rear_right"  x="${-off_x}" y="${-off_y}" roller_type="1" hub_mass="${hub_mass}" wheel_radius="${wheel_radius}"/>
   <!-- 6. ros2_control & Gazebo -->
   <xacro:arg name="gazebo" default="false"/>
@@ -137,5 +137,5 @@
       <gz_frame_id>camera_link_optical</gz_frame_id>
       <camera>
-        <horizontal_fov>1.2</horizontal_fov>
+        <horizontal_fov>2.61799</horizontal_fov>
         <image>
           <width>640</width>
