Commit message: Fix AprilTag models in Gazebo by applying PBR materials to CAD panels

File: main_ws/src/bringup/robot_bringup/urdf/include/wheel.xacro (robot description, xacro)
@@ -26,5 +26,5 @@
       <parent link="base_link"/><child link="${name}_wheel_link"/>
       <origin xyz="${x} ${y} 0" rpy="-1.57 0 0"/><axis xyz="0 0 1"/>
-      <limit effort="6.0" velocity="25.0"/>
+      <limit effort="50.0" velocity="100.0"/>
       <dynamics damping="0.1" friction="0.1"/>
     </joint>

File: main_ws/src/bringup/robot_bringup/urdf/robot.urdf.xacro (robot description, xacro)
@@ -74,5 +74,7 @@
         <joint name="${name}_wheel_joint">
           <command_interface name="velocity">
-            <param name="p">40.0</param><param name="i">1.0</param><param name="d">1.0</param>
+            <param name="p">80.0</param><param name="i">10.0</param><param name="d">2.0</param>
+            <param name="i_clamp">10.0</param>
+            <param name="max_effort">20.0</param>
           </command_interface>
           <state_interface name="position"/><state_interface name="velocity"/><state_interface name="effort"/>
@@ -93,3 +95,24 @@
     </plugin>
   </gazebo>
+  <!-- Gazebo IMU Sensor Plugin -->
+  <gazebo reference="base_link">
+    <sensor name="imu_sensor" type="imu">
+      <always_on>true</always_on>
+      <update_rate>100</update_rate>
+      <topic>/imu</topic>
+      <gz_frame_id>base_link</gz_frame_id>
+      <imu>
+        <angular_velocity>
+          <x><noise type="none"/></x>
+          <y><noise type="none"/></y>
+          <z><noise type="none"/></z>
+        </angular_velocity>
+        <linear_acceleration>
+          <x><noise type="none"/></x>
+          <y><noise type="none"/></y>
+          <z><noise type="none"/></z>
+        </linear_acceleration>
+      </imu>
+    </sensor>
+  </gazebo>
 </robot>

Commit message: Implement true physical mecanum rollers for DART physics

File: main_ws/src/bringup/robot_bringup/urdf/include/wheel.xacro (robot description, xacro)
@@ -6,13 +6,19 @@
     <xacro:property name="pos_y" value="${0.038 * sin(angle_rad)}"/>
     <xacro:property name="rot_r" value="${roller_type * pi/4}"/>
-    <joint name="${wheel_prefix}_barrel_${num}_joint" type="fixed">
+    <joint name="${wheel_prefix}_barrel_${num}_joint" type="continuous">
       <parent link="${wheel_prefix}_link"/><child link="${wheel_prefix}_barrel_${num}_link"/>
       <origin xyz="${pos_x} ${pos_y} 0" rpy="${rot_r} 0 ${angle_rad}"/>
+      <axis xyz="0 0 1"/>
+      <dynamics damping="0.001" friction="0.001"/>
     </joint>
     <link name="${wheel_prefix}_barrel_${num}_link">
+      <xacro:cylinder_inertia m="0.01" r="0.012" h="0.032"/>
       <visual name="${wheel_prefix}_barrel_${num}_vis">
         <geometry><cylinder radius="0.012" length="0.032"/></geometry>
         <material name="black"/>
       </visual>
+      <collision name="${wheel_prefix}_barrel_${num}_col">
+        <geometry><cylinder radius="0.012" length="0.032"/></geometry>
+      </collision>
     </link>
   </xacro:macro>
@@ -21,5 +27,5 @@
       <xacro:cylinder_inertia m="${hub_mass}" r="${wheel_radius}" h="0.04"/>
       <visual name="${name}_hub_vis"><geometry><cylinder radius="${wheel_radius}" length="0.04"/></geometry><material name="aluminum"/></visual>
-      <collision name="${name}_hub_col"><geometry><cylinder radius="${wheel_radius}" length="0.04"/></geometry></collision>
+      <!-- Hub collision removed to allow rollers to contact the ground -->
     </link>
     <joint name="${name}_wheel_joint" type="continuous">

Commit message: Fix wheel rollers getting stuck by using sphere collisions

File: main_ws/src/bringup/robot_bringup/urdf/include/wheel.xacro (robot description, xacro)
@@ -10,5 +10,5 @@
       <origin xyz="${pos_x} ${pos_y} 0" rpy="${rot_r} 0 ${angle_rad}"/>
       <axis xyz="0 0 1"/>
-      <dynamics damping="0.001" friction="0.001"/>
+      <dynamics damping="0.0" friction="0.0"/>
     </joint>
     <link name="${wheel_prefix}_barrel_${num}_link">
@@ -19,5 +19,5 @@
       </visual>
       <collision name="${wheel_prefix}_barrel_${num}_col">
-        <geometry><cylinder radius="0.012" length="0.032"/></geometry>
+        <geometry><sphere radius="0.012"/></geometry>
       </collision>
     </link>

Commit message: Revert physical rollers to fix physics jam and use sphere collision for fdir1 support

File: main_ws/src/bringup/robot_bringup/urdf/include/wheel.xacro (robot description, xacro)
@@ -6,19 +6,13 @@
     <xacro:property name="pos_y" value="${0.038 * sin(angle_rad)}"/>
     <xacro:property name="rot_r" value="${roller_type * pi/4}"/>
-    <joint name="${wheel_prefix}_barrel_${num}_joint" type="continuous">
+    <joint name="${wheel_prefix}_barrel_${num}_joint" type="fixed">
       <parent link="${wheel_prefix}_link"/><child link="${wheel_prefix}_barrel_${num}_link"/>
       <origin xyz="${pos_x} ${pos_y} 0" rpy="${rot_r} 0 ${angle_rad}"/>
-      <axis xyz="0 0 1"/>
-      <dynamics damping="0.0" friction="0.0"/>
     </joint>
     <link name="${wheel_prefix}_barrel_${num}_link">
-      <xacro:cylinder_inertia m="0.01" r="0.012" h="0.032"/>
       <visual name="${wheel_prefix}_barrel_${num}_vis">
         <geometry><cylinder radius="0.012" length="0.032"/></geometry>
         <material name="black"/>
       </visual>
-      <collision name="${wheel_prefix}_barrel_${num}_col">
-        <geometry><sphere radius="0.012"/></geometry>
-      </collision>
     </link>
   </xacro:macro>
@@ -27,5 +21,5 @@
       <xacro:cylinder_inertia m="${hub_mass}" r="${wheel_radius}" h="0.04"/>
       <visual name="${name}_hub_vis"><geometry><cylinder radius="${wheel_radius}" length="0.04"/></geometry><material name="aluminum"/></visual>
-      <!-- Hub collision removed to allow rollers to contact the ground -->
+      <collision name="${name}_hub_col"><geometry><sphere radius="${wheel_radius}"/></geometry></collision>
     </link>
     <joint name="${name}_wheel_joint" type="continuous">

Commit message: Restore working physical mecanum rollers. Foxglove was broken due to a node crash, not physics.

File: main_ws/src/bringup/robot_bringup/urdf/include/wheel.xacro (robot description, xacro)
@@ -6,13 +6,19 @@
     <xacro:property name="pos_y" value="${0.038 * sin(angle_rad)}"/>
     <xacro:property name="rot_r" value="${roller_type * pi/4}"/>
-    <joint name="${wheel_prefix}_barrel_${num}_joint" type="fixed">
+    <joint name="${wheel_prefix}_barrel_${num}_joint" type="continuous">
       <parent link="${wheel_prefix}_link"/><child link="${wheel_prefix}_barrel_${num}_link"/>
       <origin xyz="${pos_x} ${pos_y} 0" rpy="${rot_r} 0 ${angle_rad}"/>
+      <axis xyz="0 0 1"/>
+      <dynamics damping="0.001" friction="0.001"/>
     </joint>
     <link name="${wheel_prefix}_barrel_${num}_link">
+      <xacro:cylinder_inertia m="0.01" r="0.012" h="0.032"/>
       <visual name="${wheel_prefix}_barrel_${num}_vis">
         <geometry><cylinder radius="0.012" length="0.032"/></geometry>
         <material name="black"/>
       </visual>
+      <collision name="${wheel_prefix}_barrel_${num}_col">
+        <geometry><cylinder radius="0.012" length="0.032"/></geometry>
+      </collision>
     </link>
   </xacro:macro>
@@ -21,5 +27,5 @@
       <xacro:cylinder_inertia m="${hub_mass}" r="${wheel_radius}" h="0.04"/>
       <visual name="${name}_hub_vis"><geometry><cylinder radius="${wheel_radius}" length="0.04"/></geometry><material name="aluminum"/></visual>
-      <collision name="${name}_hub_col"><geometry><sphere radius="${wheel_radius}"/></geometry></collision>
+      <!-- Hub collision removed to allow rollers to contact the ground -->
     </link>
     <joint name="${name}_wheel_joint" type="continuous">

Commit message: Fix mecanum kinematics and apriltag camera sync

File: main_ws/src/bringup/robot_bringup/urdf/include/wheel.xacro (robot description, xacro)
@@ -18,7 +18,5 @@
         <material name="black"/>
       </visual>
-      <collision name="${wheel_prefix}_barrel_${num}_col">
-        <geometry><cylinder radius="0.012" length="0.032"/></geometry>
-      </collision>
+      <!-- Barrel collision removed to use fake mecanum physics on hub -->
     </link>
   </xacro:macro>
@@ -27,5 +25,7 @@
       <xacro:cylinder_inertia m="${hub_mass}" r="${wheel_radius}" h="0.04"/>
       <visual name="${name}_hub_vis"><geometry><cylinder radius="${wheel_radius}" length="0.04"/></geometry><material name="aluminum"/></visual>
-      <!-- Hub collision removed to allow rollers to contact the ground -->
+      <collision name="${name}_hub_col">
+        <geometry><cylinder radius="${wheel_radius}" length="0.04"/></geometry>
+      </collision>
     </link>
     <joint name="${name}_wheel_joint" type="continuous">

File: main_ws/src/bringup/robot_bringup/urdf/robot.urdf.xacro (robot description, xacro)
@@ -23,5 +23,5 @@
     <collision name="base_col"><origin xyz="0 0 0.05"/><geometry><box size="${base_l} ${base_w} ${base_h}"/></geometry></collision>
   </link>
-  <joint name="base_joint" type="fixed"><parent link="base_footprint"/><child link="base_link"/><origin xyz="0 0 0.05"/></joint>
+  <joint name="base_joint" type="fixed"><parent link="base_footprint"/><child link="base_link"/><origin xyz="0 0 ${wheel_radius}"/></joint>
   <!-- 4. Sensors -->
   <xacro:property name="imu_o" value="${props['sensors']['imu_offset']}"/>
@@ -47,8 +47,8 @@
   <xacro:property name="off_x" value="${wheel_base / 2.0}"/>
   <xacro:property name="off_y" value="${wheel_sep / 2.0}"/>
-  <xacro:mecanum_wheel name="front_left"  x="${off_x}"  y="${off_y}" roller_type="1" hub_mass="${hub_mass}" wheel_radius="${wheel_radius}"/>
-  <xacro:mecanum_wheel name="front_right" x="${off_x}"  y="${-off_y}" roller_type="-1"  hub_mass="${hub_mass}" wheel_radius="${wheel_radius}"/>
-  <xacro:mecanum_wheel name="rear_left"   x="${-off_x}" y="${off_y}"  roller_type="-1"  hub_mass="${hub_mass}" wheel_radius="${wheel_radius}"/>
-  <xacro:mecanum_wheel name="rear_right"  x="${-off_x}" y="${-off_y}" roller_type="1" hub_mass="${hub_mass}" wheel_radius="${wheel_radius}"/>
+  <xacro:mecanum_wheel name="front_left"  x="${off_x}"  y="${off_y}" roller_type="-1" hub_mass="${hub_mass}" wheel_radius="${wheel_radius}"/>
+  <xacro:mecanum_wheel name="front_right" x="${off_x}"  y="${-off_y}" roller_type="1"  hub_mass="${hub_mass}" wheel_radius="${wheel_radius}"/>
+  <xacro:mecanum_wheel name="rear_left"   x="${-off_x}" y="${off_y}"  roller_type="1"  hub_mass="${hub_mass}" wheel_radius="${wheel_radius}"/>
+  <xacro:mecanum_wheel name="rear_right"  x="${-off_x}" y="${-off_y}" roller_type="-1" hub_mass="${hub_mass}" wheel_radius="${wheel_radius}"/>
   <!-- 6. ros2_control & Gazebo -->
   <xacro:arg name="gazebo" default="false"/>
@@ -137,5 +137,5 @@
       <gz_frame_id>camera_link_optical</gz_frame_id>
       <camera>
-        <horizontal_fov>2.61799</horizontal_fov>
+        <horizontal_fov>1.2</horizontal_fov>
         <image>
           <width>640</width>

Commit message: Fix image flipping and mecanum sideways movement

File: main_ws/src/bringup/robot_bringup/urdf/include/wheel.xacro (robot description, xacro)
@@ -26,5 +26,5 @@
       <visual name="${name}_hub_vis"><geometry><cylinder radius="${wheel_radius}" length="0.04"/></geometry><material name="aluminum"/></visual>
       <collision name="${name}_hub_col">
-        <geometry><cylinder radius="${wheel_radius}" length="0.04"/></geometry>
+        <geometry><sphere radius="${wheel_radius}"/></geometry>
       </collision>
     </link>
